File: panel-tester-hardware/CTS_Solar_Panel_Load_Tester.kicad_sch (KiCad schematic)
At the start: 11 parts, among them J1 Screw_Terminal_01x02, J2 Conn_01x02_Pin, J3 Conn_01x07, U1 INA219AxD, U2 YAAJ_BluePill

Commit message: Revert "Bluepill layout edits"
This reverts commit 7404dadbf005f9dc7929b7ea0254307db19fd9e4.
Parts:
- U2: footprint BluePill:YAAJ_BluePill_2 -> (none)
Changed lines of the file:
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@@
 			)
 		)
-		(property "Footprint" "BluePill:YAAJ_BluePill_2"
+		(property "Footprint" ""
 			(at 73.025 46.99 90)
 			(effects
