File: panel-tester-hardware/CTS_Solar_Panel_Load_Tester.kicad_sch (KiCad schematic)
At the start: 29 parts, among them J1 Screw_Terminal_01x02, J2 Conn_01x02_Pin, J3 Conn_01x07, J4 Conn_01x20_Pin, J5 Conn_01x20_Pin, Q2 2N7002, U1 INA219AxD, U3 LM311

Commit message: changed solar panel connection
Connections:
- net V_SOLAR_INPUT_POS: now also RF1-1.1 (Pin_1), R_SHUNT3.2, U1.7 (IN-), U3.7; no longer R_SHUNT3.1, U1.8 (IN+)
- new net: R_SHUNT3.1, U1.8 (IN+)
Changed lines of the file:
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@@
 	)
 	(junction
-		(at 148.59 36.83)
+		(at 255.27 97.79)
+		(diameter 0)
+		(color 0 0 0 0)
+	)
+	(junction
+		(at 224.79 34.29)
 		(diameter 0)
 		(color 0 0 0 0)
@@
 	(wire
 		(pts
-			(xy 219.71 34.29) (xy 229.87 34.29)
+			(xy 219.71 34.29) (xy 224.79 34.29)
 		)
 		(stroke
@@
 	(wire
 		(pts
+			(xy 224.79 26.67) (xy 255.27 26.67)
+		)
+		(stroke
+			(width 0)
+			(type default)
+		)
+	)
+	(wire
+		(pts
 			(xy 222.25 38.1) (xy 222.25 36.83)
 		)
@@
 	(wire
 		(pts
+			(xy 255.27 26.67) (xy 255.27 97.79)
+		)
+		(stroke
+			(width 0)
+			(type default)
+		)
+	)
+	(wire
+		(pts
+			(xy 224.79 34.29) (xy 224.79 26.67)
+		)
+		(stroke
+			(width 0)
+			(type default)
+		)
+	)
+	(wire
+		(pts
 			(xy 236.22 73.66) (xy 242.57 73.66)
 		)
@@
 	(wire
 		(pts
+			(xy 255.27 97.79) (xy 255.27 109.22)
+		)
+		(stroke
+			(width 0)
+			(type default)
+		)
+	)
+	(wire
+		(pts
 			(xy 95.25 92.71) (xy 99.06 92.71)
 		)
@@
 	(wire
 		(pts
+			(xy 224.79 34.29) (xy 229.87 34.29)
+		)
+		(stroke
+			(width 0)
+			(type default)
+		)
+	)
+	(wire
+		(pts
 			(xy 123.19 92.71) (xy 127 92.71)
 		)
@@
 	(wire
 		(pts
-			(xy 148.59 31.75) (xy 148.59 36.83)
-		)
-		(stroke
-			(width 0)
-			(type default)
-		)
-	)
-	(wire
-		(pts
 			(xy 231.14 35.56) (xy 232.41 35.56)
 		)
@@
 		(pts
 			(xy 231.14 100.33) (xy 231.14 106.68)
-		)
-		(stroke
-			(width 0)
-			(type default)
-		)
-	)
-	(wire
-		(pts
-			(xy 255.27 97.79) (xy 255.27 109.22)
 		)
 		(stroke
@@
 	(global_label "V_SOLAR_INPUT_POS"
 		(shape input)
-		(at 148.59 31.75 180)
+		(at 146.05 46.99 270)
 		(fields_autoplaced yes)
 		(effects
@@
 		)
 		(property "Intersheetrefs" "${INTERSHEET_REFS}"
-			(at 126.3733 31.75 0)
+			(at 146.05 69.2067 90)
 			(effects
 				(font
